File: kicad/hack_badge.kicad_pcb (KiCad board)
At the start: 2 copper layers, 50.8 x 50.8 mm, 18 parts, among them U1 US1881EUA-AAA-000-BU, U2 US1881EUA-AAA-000-BU

Commit message: complete
Parts:
- moved R4 9.88 mm to (72.1, 58.9), turned to 0 degrees
- moved R1 9.71 mm to (80.3, 93.5), turned to 180 degrees
- moved D1 5.18 mm to (56.9, 93.5)
- moved D4 4.93 mm to (95.2, 58.9)
- moved D6 3.42 mm to (85.1, 58.9)
- moved D2 3.42 mm to (67.3, 93.5)
- moved D3 3.37 mm to (57.1, 58.9)
- moved D5 3.37 mm to (95.2, 93.5)
- moved R2 2.54 mm to (68.6, 58.9)
- moved R3 2.54 mm to (83.8, 93.5)
- moved JP1 2.16 mm to (68.3, 99.1)
- moved JP2 2.16 mm to (84.1, 53.3)
- moved C1 1.60 mm to (60.2, 97.3)
- moved C2 1.57 mm to (92.2, 55.1)
- moved U1 1.52 mm to (64.0, 98.6)
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Routing:
- net /GND: track 168.9 -> 137.4 mm
- net /R3D5: track 15.0 -> 11.7 mm
- net /R2D3: track 15.0 -> 11.8 mm
- net /R4D6: track 9.66 -> 6.85 mm
- net /R1D2: track 9.56 -> 6.85 mm
- net /BPOS: track 38.0 -> 40.1 mm
- net /A3V: track 60.8 -> 62.8 mm
- net /B3V: track 61.4 -> 63.0 mm
- net /AVDD: track 10.3 -> 11.4 mm
- net /BVDD: track 10.2 -> 11.3 mm
- net /APOS: track 39.3 -> 40.2 mm
Other:
- outline, holes or cut-outs redrawn
- board text added: "hackpgh.org"
- board text added: "if it smells like chicken you're holding it wrong !"
